File: RaspberryPi_IO-Link_Hat.kicad_sch (KiCad schematic)
At the start: 45 parts, among them J1 Jack-DC, J2 Raspberry_Pi_2_3, J3 Conn_01x03_Male, J4 Conn_01x03_Male, J5 Conn_01x03_Male, J6 Conn_01x03_Male, Q1 Q_PMOS_GSD, Q2 Q_NMOS_GSD, Q3 Q_NMOS_GSD, Q4 FQT7N10LTF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

Commit message: fix: 電流検出抵抗を 2012 サイズに変更
Parts:
- R11: Mouser 667-ERJ-3RSFR20V -> 667-ERJ-6BSFR20V
Changed lines of the file:
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@@
       (effects (font (size 1.27 1.27)) hide)
     )
-    (property "Mouser" "667-ERJ-3RSFR20V" (id 4) (at 214.63 83.82 0)
+    (property "Mouser" "667-ERJ-6BSFR20V" (id 4) (at 214.63 83.82 0)
       (effects (font (size 1.27 1.27)) hide)
     )
